File: kicad.kicad_pcb (KiCad board)
At the start: 2 copper layers, 14 parts

Commit message: OSHW logo
Parts:
- added SYM: Symbol_OSHW-Logo_CopperTop_07Jul2012, Footprint_Symbols:Symbol_OSHW-Logo_CopperTop, F.Cu at (122.2, 71.8)
Changed lines of the file:
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@@
     (links 0)
     (no_connects 0)
-    (area 0 0 0 0)
+    (area 65.816783 66.8022 125.429762 98.215128)
     (thickness 1.6)
     (drawings 9)
     (tracks 0)
     (zones 0)
-    (modules 14)
+    (modules 15)
     (nets 1)
   )
@@
   )
   (setup
-    (last_trace_width 0.31)
+    (last_trace_width 0.254)
     (user_trace_width 0.12)
     (user_trace_width 0.15)
@@
       (effects (font (size 1.00076 1.00076) (thickness 0.3048)))
     )
-    (fp_text value VAL** (at 0 3.81) (layer F.SilkS)
-      (effects (font (size 1.00076 1.00076) (thickness 0.3048)))
+    (fp_text value VAL** (at 0 3.81) (layer F.SilkS) hide
+      (effects (font (size 1.00076 1.00076) (thickness 0.25019)))
     )
     (fp_line (start -1.99136 -2.4892) (end 2.4892 -2.4892) (layer F.SilkS) (width 0.14986))
@@
     (pad 1 thru_hole circle (at 0 0) (size 4.50088 4.50088) (drill 1.99898) (layers *.Cu *.Mask F.SilkS))
   )
+  (module Footprint_Symbols:Symbol_OSHW-Logo_CopperTop (layer F.Cu)
+    (at 122.2 71.8)
+    (descr "Symbol, OSHW-Logo, Copper Top,")
+    (tags "Symbol, OSHW-Logo, Copper Top,")
+    (fp_text reference SYM (at 0.09906 -4.38912) (layer F.SilkS) hide
+      (effects (font (thickness 0.3048)))
+    )
+    (fp_text value Symbol_OSHW-Logo_CopperTop_07Jul2012 (at 0.30988 6.56082) (layer F.SilkS) hide
+      (effects (font (thickness 0.3048)))
+    )
+    (fp_line (start 1.66878 2.68986) (end 2.02946 4.16052) (layer F.Cu) (width 0.381))
+    (fp_line (start 2.02946 4.16052) (end 2.30886 3.0988) (layer F.Cu) (width 0.381))
+    (fp_line (start 2.30886 3.0988) (end 2.61874 4.17068) (layer F.Cu) (width 0.381))
+    (fp_line (start 2.61874 4.17068) (end 2.9591 2.72034) (layer F.Cu) (width 0.381))
+    (fp_line (start 0.24892 3.38074) (end 1.03886 3.37058) (layer F.Cu) (width 0.381))
+    (fp_line (start 1.03886 3.37058) (end 1.04902 3.38074) (layer F.Cu) (width 0.381))
+    (fp_line (start 1.04902 3.38074) (end 1.04902 3.37058) (layer F.Cu) (width 0.381))
+    (fp_line (start 1.08966 2.65938) (end 1.08966 4.20116) (layer F.Cu) (width 0.381))
+    (fp_line (start 0.20066 2.64922) (end 0.20066 4.21894) (layer F.Cu) (width 0.381))
+    (fp_line (start 0.20066 4.21894) (end 0.21082 4.20878) (layer F.Cu) (width 0.381))
+    (fp_line (start -0.35052 2.75082) (end -0.70104 2.66954) (layer F.Cu) (width 0.381))
+    (fp_line (start -0.70104 2.66954) (end -1.02108 2.65938) (layer F.Cu) (width 0.381))
+    (fp_line (start -1.02108 2.65938) (end -1.25984 2.86004) (layer F.Cu) (width 0.381))
+    (fp_line (start -1.25984 2.86004) (end -1.29032 3.12928) (layer F.Cu) (width 0.381))
+    (fp_line (start -1.29032 3.12928) (end -1.04902 3.37058) (layer F.Cu) (width 0.381))
+    (fp_line (start -1.04902 3.37058) (end -0.6604 3.50012) (layer F.Cu) (width 0.381))
+    (fp_line (start -0.6604 3.50012) (end -0.48006 3.66014) (layer F.Cu) (width 0.381))
+    (fp_line (start -0.48006 3.66014) (end -0.43942 3.95986) (layer F.Cu) (width 0.381))
+    (fp_line (start -0.43942 3.95986) (end -0.67056 4.18084) (layer F.Cu) (width 0.381))
+    (fp_line (start -0.67056 4.18084) (end -0.9906 4.20878) (layer F.Cu) (width 0.381))
+    (fp_line (start -0.9906 4.20878) (end -1.34112 4.09956) (layer F.Cu) (width 0.381))
+    (fp_line (start -2.37998 2.64922) (end -2.6289 2.66954) (layer F.Cu) (width 0.381))
+    (fp_line (start -2.6289 2.66954) (end -2.8702 2.91084) (layer F.Cu) (width 0.381))
+    (fp_line (start -2.8702 2.91084) (end -2.9591 3.40106) (layer F.Cu) (width 0.381))
+    (fp_line (start -2.9591 3.40106) (end -2.93116 3.74904) (layer F.Cu) (width 0.381))
+    (fp_line (start -2.93116 3.74904) (end -2.7305 4.06908) (layer F.Cu) (width 0.381))
+    (fp_line (start -2.7305 4.06908) (end -2.47904 4.191) (layer F.Cu) (width 0.381))
+    (fp_line (start -2.47904 4.191) (end -2.16916 4.11988) (layer F.Cu) (width 0.381))
+    (fp_line (start -2.16916 4.11988) (end -1.95072 3.93954) (layer F.Cu) (width 0.381))
+    (fp_line (start -1.95072 3.93954) (end -1.8796 3.4798) (layer F.Cu) (width 0.381))
+    (fp_line (start -1.8796 3.4798) (end -1.9304 3.07086) (layer F.Cu) (width 0.381))
+    (fp_line (start -1.9304 3.07086) (end -2.03962 2.78892) (layer F.Cu) (width 0.381))
+    (fp_line (start -2.03962 2.78892) (end -2.4003 2.65938) (layer F.Cu) (width 0.381))
+    (fp_line (start -1.78054 0.92964) (end -2.03962 1.49098) (layer F.Cu) (width 0.381))
+    (fp_line (start -2.03962 1.49098) (end -1.50114 2.00914) (layer F.Cu) (width 0.381))
+    (fp_line (start -1.50114 2.00914) (end -0.98044 1.7399) (layer F.Cu) (width 0.381))
+    (fp_line (start -0.98044 1.7399) (end -0.70104 1.89992) (layer F.Cu) (width 0.381))
+    (fp_line (start 0.73914 1.8796) (end 1.06934 1.6891) (layer F.Cu) (width 0.381))
+    (fp_line (start 1.06934 1.6891) (end 1.50876 2.0193) (layer F.Cu) (width 0.381))
+    (fp_line (start 1.50876 2.0193) (end 1.9812 1.52908) (layer F.Cu) (width 0.381))
+    (fp_line (start 1.9812 1.52908) (end 1.69926 1.04902) (layer F.Cu) (width 0.381))
+    (fp_line (start 1.69926 1.04902) (end 1.88976 0.57912) (layer F.Cu) (width 0.381))
+    (fp_line (start 1.88976 0.57912) (end 2.49936 0.39116) (layer F.Cu) (width 0.381))
+    (fp_line (start 2.49936 0.39116) (end 2.49936 -0.28956) (layer F.Cu) (width 0.381))
+    (fp_line (start 2.49936 -0.28956) (end 1.94056 -0.42926) (layer F.Cu) (width 0.381))
+    (fp_line (start 1.94056 -0.42926) (end 1.7399 -1.00076) (layer F.Cu) (width 0.381))
+    (fp_line (start 1.7399 -1.00076) (end 2.00914 -1.47066) (layer F.Cu) (width 0.381))
+    (fp_line (start 2.00914 -1.47066) (end 1.53924 -1.9812) (layer F.Cu) (width 0.381))
+    (fp_line (start 1.53924 -1.9812) (end 1.02108 -1.71958) (layer F.Cu) (width 0.381))
+    (fp_line (start 1.02108 -1.71958) (end 0.55118 -1.92024) (layer F.Cu) (width 0.381))
+    (fp_line (start 0.55118 -1.92024) (end 0.381 -2.46126) (layer F.Cu) (width 0.381))
+    (fp_line (start 0.381 -2.46126) (end -0.30988 -2.47904) (layer F.Cu) (width 0.381))
+    (fp_line (start -0.30988 -2.47904) (end -0.5207 -1.9304) (layer F.Cu) (width 0.381))
+    (fp_line (start -0.5207 -1.9304) (end -0.9398 -1.76022) (layer F.Cu) (width 0.381))
+    (fp_line (start -0.9398 -1.76022) (end -1.49098 -2.02946) (layer F.Cu) (width 0.381))
+    (fp_line (start -1.49098 -2.02946) (end -2.00914 -1.50114) (layer F.Cu) (width 0.381))
+    (fp_line (start -2.00914 -1.50114) (end -1.76022 -0.96012) (layer F.Cu) (width 0.381))
+    (fp_line (start -1.76022 -0.96012) (end -1.9304 -0.48006) (layer F.Cu) (width 0.381))
+    (fp_line (start -1.9304 -0.48006) (end -2.47904 -0.381) (layer F.Cu) (width 0.381))
+    (fp_line (start -2.47904 -0.381) (end -2.4892 0.32004) (layer F.Cu) (width 0.381))
+    (fp_line (start -2.4892 0.32004) (end -1.9304 0.5207) (layer F.Cu) (width 0.381))
+    (fp_line (start -1.9304 0.5207) (end -1.7907 0.91948) (layer F.Cu) (width 0.381))
+    (fp_line (start 0.35052 0.89916) (end 0.65024 0.7493) (layer F.Cu) (width 0.381))
+    (fp_line (start 0.65024 0.7493) (end 0.8509 0.55118) (layer F.Cu) (width 0.381))
+    (fp_line (start 0.8509 0.55118) (end 1.00076 0.14986) (layer F.Cu) (width 0.381))
+    (fp_line (start 1.00076 0.14986) (end 1.00076 -0.24892) (layer F.Cu) (width 0.381))
+    (fp_line (start 1.00076 -0.24892) (end 0.8509 -0.59944) (layer F.Cu) (width 0.381))
+    (fp_line (start 0.8509 -0.59944) (end 0.39878 -0.94996) (layer F.Cu) (width 0.381))
+    (fp_line (start 0.39878 -0.94996) (end -0.0508 -1.00076) (layer F.Cu) (width 0.381))
+    (fp_line (start -0.0508 -1.00076) (end -0.44958 -0.89916) (layer F.Cu) (width 0.381))
+    (fp_line (start -0.44958 -0.89916) (end -0.8509 -0.55118) (layer F.Cu) (width 0.381))
+    (fp_line (start -0.8509 -0.55118) (end -1.00076 -0.09906) (layer F.Cu) (width 0.381))
+    (fp_line (start -1.00076 -0.09906) (end -0.94996 0.39878) (layer F.Cu) (width 0.381))
+    (fp_line (start -0.94996 0.39878) (end -0.70104 0.70104) (layer F.Cu) (width 0.381))
+    (fp_line (start -0.70104 0.70104) (end -0.35052 0.89916) (layer F.Cu) (width 0.381))
+    (fp_line (start -0.35052 0.89916) (end -0.70104 1.89992) (layer F.Cu) (width 0.381))
+    (fp_line (start 0.35052 0.89916) (end 0.7493 1.89992) (layer F.Cu) (width 0.381))
+  )
   (gr_text "1206\n" (at 123.4 87.4) (layer F.Cu)
     (effects (font (size 1 1) (thickness 0.25)))
@@
     (effects (font (size 1 1) (thickness 0.25)))
   )
-  (gr_text QFN24 (at 114.6 77.8) (layer F.Cu)
-    (effects (font (size 1 1) (thickness 0.25)))
-  )
+  (gr_text QFN24 (at 114.6 76.2) (layer F.Cu)
+    (effects (font (size 1 1) (thickness 0.25)))
+  )
